File: sao-petal.kicad_sch (KiCad schematic)
At the start: 64 parts, among them J1 SAO CONNECTOR, U1 AS1115-BSST

Commit message: added detail image for discrepancy at test points
Parts:
- J1: footprint .sao-petal:SAO_PIN_HEADER_2x03 -> .sao-petal:SAO_PIN_HEADER_2x03_PETAL
Changed lines of the file:
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@@
 			)
 		)
-		(property "Footprint" ".sao-petal:SAO_PIN_HEADER_2x03"
+		(property "Footprint" ".sao-petal:SAO_PIN_HEADER_2x03_PETAL"
 			(at 69.215 153.67 0)
 			(effects
